File: kicad/Precision23.kicad_pcb (KiCad board)
At the start: 2 copper layers, 76.2 x 76.2 mm, 153 parts, among them J503 STANDOFF, J504 STANDOFF, J505 STANDOFF, J506 STANDOFF, U001 74HC595, U002 74HC595, U101 74HC595, U102 74HC595, U401 ATmega32U4-A, U501 SAM-M8Q, U601 TCR2EF 3.3V, Y401 16MHz

Commit message: Lots of stuff
Parts:
- removed C001, C002, C101, C102: 100nF, Capacitor_SMD:C_0603_1608Metric
- removed R001, R002, R101, R102: RP4, KwanSystems:R_Array_Convex_4x0402
- removed U001, U002, U101, U102: 74HC595, Package_SO:TSSOP-16_4.4x5mm_P0.65mm
- added J001: Conn_01x04_Pin, Connector_PinHeader_2.54mm:PinHeader_1x04_P2.54mm_Vertical, B.Cu at (92.7, 73.7)
- added J002: Conn_01x04_Pin, Connector_PinHeader_2.54mm:PinHeader_1x04_P2.54mm_Vertical, B.Cu at (92.7, 76.2)
- added J003: Conn_01x06, Connector_PinHeader_2.54mm:PinHeader_1x06_P2.54mm_Vertical, B.Cu at (71.1, 82.5)
- added J004: Conn_01x06, Connector_PinSocket_2.54mm:PinSocket_1x06_P2.54mm_Vertical, B.Cu at (101.6, 82.5)
- added J005: Conn_01x06, Connector_PinHeader_2.54mm:PinHeader_1x06_P2.54mm_Vertical, B.Cu at (68.6, 82.5)
- added J405: Conn_01x08, Connector_PinHeader_2.54mm:PinHeader_1x08_P2.54mm_Vertical, B.Cu at (80.0, 69.1)
- added J406: Conn_01x08, Connector_PinHeader_2.54mm:PinHeader_1x08_P2.54mm_Vertical, B.Cu at (97.8, 108.7)
- added R201: 68, KwanSystems:R_Array_Convex_4x0402, F.Cu at (97.8, 105.7)
- added R202: 68, KwanSystems:R_Array_Convex_4x0402, F.Cu at (80.0, 105.7)
- added R203: 68, KwanSystems:R_Array_Convex_4x0402, F.Cu at (80.0, 72.1)
- added R204: 68, KwanSystems:R_Array_Convex_4x0402, F.Cu at (97.8, 72.1)
- D000, D001, D002, D003, D004, D005, D006, D007, D008, D009, D010, D011, D012, D013, D014, D015, D016, D017, D018, D019, D020, D021, D022, D023, D024, D025, D026, D027, D028, D029, D030, D031, D032, D033, D034, D035, D036, D037, D038, D039, D040, D041, D042, D043, D044, D045, D046, D047, D048, D049, D050, D051, D052, D053, D054, D055, D056, D057, D058, D059: footprint LED_SMD:LED_0603_1608Metric -> KwanSystems:LED-0603-AC
- D100, D101, D102, D103, D104, D105, D106, D107, D108, D109, D110, D111, D112, D113, D114, D115, D116, D117, D118, D119, D120, D121, D122, D123, D124, D125, D126, D127, D128, D129, D130, D131, D132, D133, D134, D135, D136, D137, D138, D139, D140, D141, D142, D143, D144, D145, D146, D147, D148, D149, D150, D151, D152, D153, D154, D155, D156, D157, D158, D159: footprint KwanSystems:D_KINGBRIGHT_DOME -> KwanSystems:D_KINGBRIGHT_DOME_AC
- R413: footprint Resistor_SMD:R_0402_1005Metric -> Resistor_SMD:R_0603_1608Metric
- moved G101 101.6 mm to (190.5, 88.9)
- moved R403 57.7 mm to (80.0, 86.8)
- moved R413 54.7 mm to (83.6, 97.8), turned to -90 degrees
- moved R408 29.6 mm to (73.9, 89.7), turned to 0 degrees
- moved D401 23.4 mm to (77.2, 88.9), turned to 0 degrees
- moved D402 22.8 mm to (77.2, 90.4), turned to 0 degrees
- moved C601 21.0 mm to (91.9, 79.2), turned to 90 degrees
- moved S413 19.6 mm to (88.9, 101.6), turned to 180 degrees
- moved U601 16.8 mm to (88.9, 79.2), turned to 180 degrees
- moved C416 16.0 mm to (85.1, 97.8), turned to -90 degrees
- moved Y401 14.7 mm to (88.1, 97.8)
- moved C417 14.3 mm to (91.2, 97.8), turned to -90 degrees
- moved C605 12.5 mm to (85.9, 79.2), turned to 90 degrees
- moved C406 12.2 mm to (80.5, 88.9)
- moved C442 8.76 mm to (81.5, 80.3), turned to 90 degrees
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Connections:
- net /Controller/D10 renamed /D10
- net /Controller/D12 renamed /D12
- net /Controller/D17 renamed /D17
- net Net-(U401-~{RESET}) renamed /~{RESET}
- R403 pad 1: /Controller/D+ -> /Controller/D-
- R403 pad 2: /Controller/D- -> /Controller/D+
- R403 pad 3: /Controller/Q_D- -> /Controller/Q_D+
- R403 pad 4: /Controller/Q_D+ -> /Controller/Q_D-
- U401 pad 1: /Controller/D7 -> /D7
- U401 pad 10: /Controller/D16 -> /D16
- U401 pad 11: /Controller/D14 -> /D14
- U401 pad 12: /Controller/D11 -> /D11
- U401 pad 18: /Controller/D3 -> /D3
- U401 pad 19: /Controller/D2 -> /D2
- U401 pad 25: /Controller/D4 -> /D4
- U401 pad 27: /Controller/D6 -> /D6
- U401 pad 28: /Controller/D8 -> /D8
- U401 pad 29: /Controller/D9 -> /D9
- U401 pad 31: /Controller/D5 -> /D5
- U401 pad 32: /Controller/D13 -> /D13
- U401 pad 36: /Controller/A0 -> /A0
- U401 pad 37: /Controller/A1 -> /A1
- U401 pad 38: /Controller/A2 -> /A2
- U401 pad 39: /Controller/A3 -> /A3
- U401 pad 40: /Controller/A4 -> /A4
- U401 pad 41: /Controller/A5 -> /A5
- U401 pad 9: /Controller/D15 -> /D15
Routing:
- net /Charlieplex/Q16: track 0.00 -> 330.6 mm, vias 0 -> 19
- net /Charlieplex/Q14: track 0.00 -> 320.8 mm, vias 0 -> 19
- net /Charlieplex/Q15: track 0.00 -> 320.8 mm, vias 0 -> 18
- net /Charlieplex/Q13: track 0.00 -> 313.1 mm, vias 0 -> 19
- net /Charlieplex/Q12: track 0.00 -> 310.8 mm, vias 0 -> 20
- net /Charlieplex/Q10: track 0.00 -> 309.0 mm, vias 0 -> 22
- net /Charlieplex/Q11: track 0.00 -> 307.9 mm, vias 0 -> 21
- net /Charlieplex/Q09: track 0.00 -> 297.9 mm, vias 0 -> 21
- net /Charlieplex/Q06: track 0.00 -> 295.8 mm, vias 0 -> 22
- net /Charlieplex/Q07: track 0.00 -> 295.7 mm, vias 0 -> 21
- net /Charlieplex/Q08: track 0.00 -> 293.7 mm, vias 0 -> 21
- net /Charlieplex/Q05: track 0.00 -> 293.3 mm, vias 0 -> 21
- net /Charlieplex/Q04: track 0.00 -> 288.9 mm, vias 0 -> 20
- net /Charlieplex/Q03: track 0.00 -> 280.6 mm, vias 0 -> 18
- net /Charlieplex/Q02: track 0.00 -> 274.8 mm, vias 0 -> 17
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Other:
- board text added: "D+"
- board text added: "D-"
- board text added: "GND"
- board text added: "VCC"
- board text added: "black"
- board text added: "green"
- board text added: "red"
- board text added: "white"
