File: kicad/Precision23.kicad_sch (KiCad schematic)
At the start: 8 parts, among them J501 Conn_01x04_Pin, J502 Conn_01x04_Pin, J503 STANDOFF, J504 STANDOFF, J505 STANDOFF, J506 STANDOFF, U501 SAM-M8Q

Commit message: Lots of stuff
Parts:
- added J003, J005: Conn_01x06, Connector_PinHeader_2.54mm:PinHeader_1x06_P2.54mm_Vertical, symbol Connector_Generic:Conn_01x06
- added J004: Conn_01x06, Connector_PinSocket_2.54mm:PinSocket_1x06_P2.54mm_Vertical, symbol Connector_Generic:Conn_01x06
- J001: renamed from J501; footprint Connector_PinHeader_2.54mm:PinHeader_1x04_P2.54mm_Vertical_SMD_Pin1Right -> Connector_PinHeader_2.54mm:PinHeader_1x04_P2.54mm_Vertical; symbol Connector:Conn_01x04_Pin -> Connector_Generic:Conn_01x04
- J002: renamed from J502; footprint (none) -> Connector_PinHeader_2.54mm:PinHeader_1x04_P2.54mm_Vertical; symbol Connector:Conn_01x04_Pin -> Connector_Generic:Conn_01x04
Connections:
- net +3V3: now also J003.2 (Pin_2), J004.4 (Pin_4), J004.5 (Pin_5), J005.2 (Pin_2)
- net D10: now also J004.6 (Pin_6)
- net D14: now also J003.5 (Pin_5), J005.5 (Pin_5)
- net D15: now also J003.4 (Pin_4), J005.4 (Pin_4)
- net D16: now also J003.6 (Pin_6), J005.6 (Pin_6)
- net GND: now also J003.3 (Pin_3), J004.3 (Pin_3), J005.3 (Pin_3)
- net GPS_RX: now also J004.1 (Pin_1)
- net GPS_TX: now also J004.2 (Pin_2)
- new net ~{RESET}: J003.1 (Pin_1), J005.1 (Pin_1)
- no-connect marks 18 -> 8
Other:
- removed sheet Hour hand
- removed sheet Minute hand
- removed sheet Second hand
- removed sheet Third hand
- added sheet Charlieplex (charlieplex.kicad_sch)
- sheet Controller ports: added ~{RESET}; removed none
- note added: "ICSP1/MISO/"
- note added: "ICSP2"
- note added: "ICSP3/SCK/"
- note added: "ICSP4/MOSI/"
- note added: "ICSP5"
- note added: "ICSP6"
